File: schematic/NCL501/NCL501.kicad_pcb (KiCad board)
At the start: 2 copper layers, 135 x 97.8 mm, 42 parts, among them CN1 SCSI Intern, J1 SCSI extern, J2 Bus_ISA_8bit, J4 DACK/DRQ, U1 74LS175, U10 PAL16L8, U11 MIC5219-2.85YM5, U2 74LS125, U3 74LS14, U4 6116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

Commit message: Schematic updated
Parts:
- RP2, RP3, RP4: value 330E -> 220E/330E
Changed lines of the file:
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@@
     (property "Sheetfile" "NCL501.kicad_sch")
     (property "Sheetname" "")
-    (property "ki_description" "7 resistor network, star topology, bussed resistors, small symbol")
-    (property "ki_keywords" "R network star-topology")
+    (property "ki_description" "6 voltage divider network, dual terminator, SIP package")
+    (property "ki_keywords" "R network divider topology")
     (attr through_hole)
     (fp_text reference "RP2" (at 0 2.286 -90) (layer "F.SilkS")
         (effects (font (size 1 1) (thickness 0.15)))
     )
-    (fp_text value "330E" (at 10.16 2.4 90) (layer "F.Fab") hide
+    (fp_text value "220E/330E" (at 10.16 2.4 90) (layer "F.Fab") hide
         (effects (font (size 1 1) (thickness 0.15)))
     )
@@
       (stroke (width 0.1) (type solid)) (layer "F.Fab"))
     (pad "1" thru_hole rect (at 0 0 270) (size 1.6 1.6) (drill 0.8) (layers "*.Cu" "*.Mask")
-      (net 2 "GND") (pinfunction "common") (pintype "passive"))
+      (net 2 "GND") (pinfunction "COM1") (pintype "passive"))
     (pad "2" thru_hole oval (at 2.54 0 270) (size 1.6 1.6) (drill 0.8) (layers "*.Cu" "*.Mask")
       (net 24 "/SD0") (pinfunction "R1") (pintype "passive"))
@@
       (net 19 "/SD5") (pinfunction "R6") (pintype "passive"))
     (pad "8" thru_hole oval (at 17.78 0 270) (size 1.6 1.6) (drill 0.8) (layers "*.Cu" "*.Mask")
-      (net 5 "+5P") (pinfunction "R7") (pintype "passive"))
+      (net 5 "+5P") (pinfunction "COM2") (pintype "passive"))
     (model "${KICAD6_3DMODEL_DIR}/Resistor_THT.3dshapes/R_Array_SIP8.wrl"
       (offset (xyz 0 0 0))
@@
     (property "Sheetfile" "NCL501.kicad_sch")
     (property "Sheetname" "")
-    (property "ki_description" "7 resistor network, star topology, bussed resistors, small symbol")
-    (property "ki_keywords" "R network star-topology")
+    (property "ki_description" "6 voltage divider network, dual terminator, SIP package")
+    (property "ki_keywords" "R network divider topology")
     (attr through_hole)
     (fp_text reference "RP3" (at -2.54 -0.127 -180) (layer "F.SilkS")
         (effects (font (size 1 1) (thickness 0.15)))
     )
-    (fp_text value "330E" (at 10.16 2.4 90) (layer "F.Fab") hide
+    (fp_text value "220E/330E" (at 10.16 2.4 90) (layer "F.Fab") hide
         (effects (font (size 1 1) (thickness 0.15)))
     )
@@
       (stroke (width 0.1) (type solid)) (layer "F.Fab"))
     (pad "1" thru_hole rect (at 0 0 270) (size 1.6 1.6) (drill 0.8) (layers "*.Cu" "*.Mask")
-      (net 2 "GND") (pinfunction "common") (pintype "passive"))
+      (net 2 "GND") (pinfunction "COM1") (pintype "passive"))
     (pad "2" thru_hole oval (at 2.54 0 270) (size 1.6 1.6) (drill 0.8) (layers "*.Cu" "*.Mask")
       (net 18 "/SD6") (pinfunction "R1") (pintype "passive"))
@@
       (net 8 "/~{SACK}") (pinfunction "R6") (pintype "passive"))
     (pad "8" thru_hole oval (at 17.78 0 270) (size 1.6 1.6) (drill 0.8) (layers "*.Cu" "*.Mask")
-      (net 5 "+5P") (pinfunction "R7") (pintype "passive"))
+      (net 5 "+5P") (pinfunction "COM2") (pintype "passive"))
     (model "${KICAD6_3DMODEL_DIR}/Resistor_THT.3dshapes/R_Array_SIP8.wrl"
       (offset (xyz 0 0 0))
@@
     (property "Sheetfile" "NCL501.kicad_sch")
     (property "Sheetname" "")
-    (property "ki_description" "7 resistor network, star topology, bussed resistors, small symbol")
-    (property "ki_keywords" "R network star-topology")
+    (property "ki_description" "6 voltage divider network, dual terminator, SIP package")
+    (property "ki_keywords" "R network divider topology")
     (attr through_hole)
     (fp_text reference "RP4" (at -2.413 -0.127 -180) (layer "F.SilkS")
         (effects (font (size 1 1) (thickness 0.15)))
     )
-    (fp_text value "330E" (at 0.254 2.54 90) (layer "F.Fab") hide
+    (fp_text value "220E/330E" (at 0.254 2.54 90) (layer "F.Fab") hide
         (effects (font (size 1 1) (thickness 0.15)))
     )
@@
       (stroke (width 0.1) (type solid)) (layer "F.Fab"))
     (pad "1" thru_hole rect (at 0 0 270) (size 1.6 1.6) (drill 0.8) (layers "*.Cu" "*.Mask")
-      (net 2 "GND") (pinfunction "common") (pintype "passive"))
+      (net 2 "GND") (pinfunction "COM1") (pintype "passive"))
     (pad "2" thru_hole oval (at 2.54 0 270) (size 1.6 1.6) (drill 0.8) (layers "*.Cu" "*.Mask")
       (net 9 "/~{SRST}") (pinfunction "R1") (pintype "passive"))
@@
       (net 14 "/~{SIO}") (pinfunction "R6") (pintype "passive"))
     (pad "8" thru_hole oval (at 17.78 0 270) (size 1.6 1.6) (drill 0.8) (layers "*.Cu" "*.Mask")
-      (net 5 "+5P") (pinfunction "R7") (pintype "passive"))
+      (net 5 "+5P") (pinfunction "COM2") (pintype "passive"))
     (model "${KICAD6_3DMODEL_DIR}/Resistor_THT.3dshapes/R_Array_SIP8.wrl"
       (offset (xyz 0 0 0))
@@
     (effects (font (size 1 1) (thickness 0.1)) (justify left bottom))
   )
+  (dimension (type aligned) (layer "Dwgs.User")
+    (pts (xy 252.25 151.25) (xy 252.25 53.5))
+    (height 14)
+    (gr_text "97,7500 mm" (at 265.1 102.375 90) (layer "Dwgs.User")
+      (effects (font (size 1 1) (thickness 0.15)))
+    )
+    (format (prefix "") (suffix "") (units 3) (units_format 1) (precision 4))
+    (style (thickness 0.1) (arrow_length 1.27) (text_position_mode 0) (extension_height 0.58642) (extension_offset 0.5) keep_text_aligned)
+  )
+  (dimension (type aligned) (layer "Dwgs.User")
+    (pts (xy 252.25 53.5) (xy 117.25 53.5))
+    (height 4.731999)
+    (gr_text "135,0000 mm" (at 184.75 47.618001) (layer "Dwgs.User")
+      (effects (font (size 1 1) (thickness 0.15)))
+    )
+    (format (prefix "") (suffix "") (units 3) (units_format 1) (precision 4))
+    (style (thickness 0.1) (arrow_length 1.27) (text_position_mode 0) (extension_height 0.58642) (extension_offset 0.5) keep_text_aligned)
+  )
+  (dimension (type aligned) (layer "Dwgs.User")
+    (pts (xy 252.25 53.5) (xy 252.25 143.25))
+    (height -10.386)
+    (gr_text "89,7500 mm" (at 261.486 98.375 90) (layer "Dwgs.User")
+      (effects (font (size 1 1) (thickness 0.15)))
+    )
+    (format (prefix "") (suffix "") (units 3) (units_format 1) (precision 4))
+    (style (thickness 0.1) (arrow_length 1.27) (text_position_mode 0) (extension_height 0.58642) (extension_offset 0.5) keep_text_aligned)
+  )
   (segment (start 153.67 111.76) (end 155.194 110.236) (width 1) (layer "F.Cu") (net 1))
