File: schematic/NCL501/untitled.kicad_sch (KiCad schematic)
At the start: 15 parts, among them U2 74LS125, U3 74LS14

Commit message: first manufactured Version
Connections:
- net GND: now also U2.1, U2.2, U3.1, U3.11, U3.3, U3.9
Other:
- note removed: "are these not connected?"
- moved on the sheet: U2A, U3B, U3D, U3E
